File: KiCad PCB files - BASIC2/VectorScopeMusicAddon.kicad_pcb (KiCad board)
At the start: 2 copper layers, 37.5 x 24 mm, 14 parts, among them J1 Conn_01x09_Socket, J3 AudioJack3_SwitchTR, SW2 SW_Push_DPDT, U1 OPA2192

Commit message: basic2 fonts
Parts:
- added Ref**: Val**, davedarko:davedarko_logo_silk_outline, F.Cu at (5.00, 19.5)
- added Ref**: Val**, davedarko:davedarko_logo_silk_outline, B.Cu at (16.0, 4.40)
Routing:
- net right_in: track 17.1 -> 15.2 mm
Other:
- board text added: "https://github.com/davedarko /VectorScopeMusicAddon vectorscope Badge Addon for Oscilloscope Music @davedarko 2024/09 compatible with badges: Supercon 2023 | Europe 2024"
- board text added: "left | x-channel | tip right | y-channel | ring"
- board text removed: "https://github.com/davedarko /VectorScopeMusicAddon Hackaday Badge Addon Oscilloscope Music @davedarko 2024/09 compatible with badges: Supercon 2022 | Europe 2023"
- board text removed: "left | x-channel | tip"
- board text removed: "right | y-channel | ring"
